File: VWS_SDR.kicad_sch (KiCad schematic)
At the start: 102 parts, among them J1 RF_IN, J2 IQ_Out, J3 Si5351 Socket, J4 IF Breakout, J5 GPIO Breakout, J6 I2C Breakout, J7 SWD, J8 GPIO Breakout, J9 Power Breakout, U1 GALI-S66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

Commit message: Update pins used on pico
Parts:
- added J10: UART, Connector_PinHeader_2.54mm:PinHeader_1x03_P2.54mm_Vertical, symbol Connector:Conn_01x03_Pin
- R26, R27: value 330 -> 680
Connections:
- net GND: now also J10.3 (Pin_3)
- net SCL: now also U5.7 (GPIO5); no longer U5.2 (GPIO1)
- net SDA: now also U5.6 (GPIO4); no longer U5.1 (GPIO0)
- new net UART0 RX: J10.2 (Pin_2), U5.2 (GPIO1)
- new net UART0 TX: J10.1 (Pin_1), U5.1 (GPIO0)
- no-connect marks 11 -> 9
Other:
- moved on the sheet: D3, D4, J7, R28, R29
